File: kicad/parasite.kicad_pcb (KiCad board)
At the start: 2 copper layers, 22 x 126.4 mm, 31 parts, among them Q1 MMBT3906, Q4 Q_Photo_NPN, SW1 B3U-1000P, U1 E73-2G4M08S1C, U2 SHTC3, Y1 32.768kHz

Commit message: Ryan changes
Parts:
- removed C3, C4: 12p, Capacitor_SMD:C_0402_1005Metric
- removed Y1: 32.768kHz, Crystal:Crystal_SMD_3215-2Pin_3.2x1.5mm
- added D5: 1N5819WS, Diode_SMD:D_SOD-323, F.Cu at (68.0, 48.4)
- added J1: USB_C_Receptacle_USB2.0, Connector_USB:USB_C_Receptacle_HRO_TYPE-C-31-M-12, B.Cu at (68.0, 34.2)
- added J4: Programmer, plumtwisttester:j2thing, B.Cu at (74.4, 42.1)
- added Q2: Q_PMOS_SGD, Package_TO_SOT_SMD:SOT-23, F.Cu at (68.0, 51.2)
- added R3: 5k1, Resistor_SMD:R_0402_1005Metric, F.Cu at (66.1, 53.6)
- added R5: 5k1, Resistor_SMD:R_0402_1005Metric, F.Cu at (69.9, 53.6)
- added R9: 10k, Resistor_SMD:R_0402_1005Metric, F.Cu at (68.0, 53.6)
- RST1, SW1: footprint snapeda:SW_B3U-1000P -> lemonlib:SW_Push_SPST_NO_Xunpu
- U1: value E73-2G4M08S1C -> ~; footprint snapeda:E73-2G4M08S1C -> lemonlib:XCVR_MS88SF2
- moved R10 2.73 mm to (58.0, 32.5), turned to -90 degrees
- moved Q4 2.14 mm to (57.8, 34.8)
- moved U1 1.42 mm to (68.0, 35.6)
- moved TP3 0.74 mm to (78.1, 39.8)
- moved TP1 0.72 mm to (78.1, 34.7)
- moved TP2 0.72 mm to (78.1, 37.2)
- moved TP4 0.72 mm to (78.1, 42.3)
- moved TP7 0.72 mm to (78.1, 32.2)
- moved TP8 0.72 mm to (78.1, 29.6)
- moved RST1 0.35 mm to (72.0, 50.2)
- moved SW1 0.13 mm to (64.0, 50.2)
Connections:
- BT1 pad 1: +3V0 -> VBAT
- C2 pad 1: +3V0 -> VDD
- R7 pad 2: +3V0 -> VDD
- R8 pad 1: +3V0 -> VDD
- TP7 pad 1: +3V0 -> VDD
- U1 pad 1: unconnected-(U1C-P1.11-Pad1) -> GND
- U1 pad 10: BTN1 -> PWM
- U1 pad 11: Net-(U1B-P0.00/XL1) -> LED
- U1 pad 12: unconnected-(U1B-P0.26-Pad12) -> BTN1
- U1 pad 13: Net-(U1B-P0.01/XL2) -> GND
- U1 pad 14: unconnected-(U1B-P0.06-Pad14) -> VDD
- U1 pad 15: PWM -> VIN
- U1 pad 16: unconnected-(U1B-P0.08-Pad16) -> D_N
- U1 pad 17: unconnected-(U1C-P1.09-Pad17) -> D_P
- U1 pad 18: unconnected-(U1B-P0.04/AIN2-Pad18) -> SCL
- U1 pad 19: +3V0 -> SDA
- U1 pad 20: unconnected-(U1B-P0.12-Pad20) -> RST
- U1 pad 21: GND -> unconnected-(U1-P0.20*-Pad21)
- U1 pad 23: +3V0 -> unconnected-(U1-P0.24*-Pad23)
- U1 pad 25: unconnected-(U1A-DCCH-Pad25) -> SWDIO
- U1 pad 26: RST -> SWDCLK
- U1 pad 28: unconnected-(U1B-P0.15-Pad28) -> 0.10
- U1 pad 3: SENS_OUT -> unconnected-(U1-P1.15-Pad3)
- U1 pad 4: LED -> PHOTO_V
- U1 pad 5: GND -> PHOTO_OUT
- U1 pad 7: PHOTO_OUT -> SENS_OUT
- U1 pad 8: PHOTO_V -> unconnected-(U1-P0.04*A-Pad8)
- U2 pad 1: +3V0 -> VDD
Routing:
- net VDD: track 0.00 -> 84.9 mm, vias 0 -> 6
- net +3V0: track 76.5 -> 0.00 mm, vias 8 -> 0
- net GND: track 22.2 -> 56.6 mm, vias 29 -> 32
- net D_P: track 0.00 -> 27.3 mm, vias 0 -> 1
- net VBUS: track 0.00 -> 25.9 mm, vias 0 -> 2
- net D_N: track 0.00 -> 24.8 mm, vias 0 -> 1
- net /CC2: track 0.00 -> 22.8 mm, vias 0 -> 3
- net /CC1: track 0.00 -> 20.5 mm, vias 0 -> 1
- net RST: track 11.9 -> 25.1 mm, vias 2 -> 1
- net VIN: track 0.00 -> 12.7 mm
- net Net-(U1B-P0.01/XL2): track 11.1 -> 0.00 mm
- net VBAT: track 0.00 -> 11.1 mm, vias 0 -> 1
- net Net-(U1B-P0.00/XL1): track 10.2 -> 0.00 mm
- net SWDCLK: track 6.42 -> 16.1 mm, vias 2 -> 3
- net SCL: track 22.2 -> 15.6 mm
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Other:
- outline, holes or cut-outs redrawn
- rule pad_to_mask_clearance: 0.051 -> 0
- board text added: "GND"
- board text added: "RST"
- board text added: "SW1"
- board text added: "SWDCLK"
- board text added: "SWDIO"
- board text added: "VDD"
- board text added: "b-parasite 2.0.0ry1 rbaron.net"
- board text added: "with mods by Ryan"
- board text removed: "JLCJLCJLCJLC"
- board text removed: "b-parasite 2.0.0 rbaron.net"
