File: kicad/parasite.kicad_sch (KiCad schematic)
At the start: 29 parts, among them Q1 MMBT3906, Q4 Q_Photo_NPN, SW1 B3U-1000P, U1 E73-2G4M08S1C, U2 SHTC3, Y1 32.768kHz

Commit message: Ryan changes
Parts:
- removed C3, C4: 12p, Capacitor_SMD:C_0402_1005Metric, symbol Device:C_Small
- removed U1: E73-2G4M08S1C, snapeda:E73-2G4M08S1C, symbol E73:E73-2G4M08S1C
- removed Y1: 32.768kHz, Crystal:Crystal_SMD_3215-2Pin_3.2x1.5mm, symbol Device:Crystal
- added D5: 1N5819WS, Diode_SMD:D_SOD-323, symbol Diode:1N5819WS
- added J1: USB_C_Receptacle_USB2.0, Connector_USB:USB_C_Receptacle_HRO_TYPE-C-31-M-12, symbol Connector:USB_C_Receptacle_USB2.0_16P
- added J4: Programmer, plumtwisttester:j2thing, symbol Connector_Generic:Conn_02x03_Top_Bottom
- added Q2: Q_PMOS_SGD, Package_TO_SOT_SMD:SOT-23, symbol Device:Q_PMOS_GSD
- added R3, R5: 5k1, Resistor_SMD:R_0402_1005Metric, symbol Device:R_Small
- added R9: 10k, Resistor_SMD:R_0402_1005Metric, symbol Device:R_Small_US
- added U1: (no value), lemonlib:XCVR_MS88SF2, symbol lemonlib:nRF52840-MS88SF21
- R2: Field5 (none) -> ${REFERENCE}
- RST1, SW1: footprint SW_B3U-1000P -> lemonlib:SW_Push_SPST_NO_Xunpu; DESCRIPTION Tactile Switch SPST-NO Top Actuated Surface Mount -> (none); LCSC C231329 -> C720477
- U2: LCSC C194656 -> C54946588
Connections:
- net 0.10: now also U1.28 (P0.10)
- net BTN1: now also U1.12 (P0.12*)
- net GND: now also J1.A1 (GND), J1.A12 (GND), J1.B1 (GND), J1.B12 (GND), J1.S1 (SHIELD), J4.6 (Pin_6), R3.2, R5.2, R9.2, U1.1 (GND), U1.13 (GND)
- net LED: now also U1.11 (P1.09*)
- net PHOTO_OUT: now also U1.5 (P0.29A)
- net PHOTO_V: now also U1.4 (P0.02)
- net PWM: now also U1.10 (P0.08*)
- net RST: now also J4.3 (Pin_3), U1.20 (P0.18)
- net SCL: now also U1.18 (P0.13*)
- net SDA: now also U1.19 (P0.15*)
- net SENS_OUT: now also U1.8 (P0.04*A)
- net SWDCLK: now also J4.2 (Pin_2), U1.26 (SWCLK)
- net SWDIO: now also J4.5 (Pin_5), U1.25 (SWDIO)
- net +3V0 renamed VDD
- net VDD: now also J4.4 (Pin_4), U1.14 (VDD); no longer BT1.1 (+)
- new net CC1: J1.A5 (CC1), R3.1
- new net CC2: J1.B5 (CC2), R5.1
- new net D_N: J1.A7 (D-), J1.B7 (D-), U1.16 (D-)
- new net D_P: J1.A6 (D+), J1.B6 (D+), U1.17 (D+)
- new net VBAT: BT1.1 (+), Q2.3 (D)
- new net VBUS: D5.2 (A), J1.A4 (VBUS), J1.A9 (VBUS), J1.B4 (VBUS), J1.B9 (VBUS), Q2.1 (G), R9.1
- new net VIN: D5.1 (K), Q2.2 (S), U1.15 (VDDH)
- no-connect marks 25 -> 4
