File: kicad/parasite.kicad_sch (KiCad schematic)
At the start: 33 parts, among them J1 USB_C_Receptacle_USB2.0, J4 Programmer, Q1 MMBT3906, Q2 Q_PMOS_SGD, Q4 Q_Photo_NPN, SW1 B3U-1000P, U2 SHTC3

Commit message: Fix CI and schematic pdf
Other:
- note added: "USB power and data"
- moved on the sheet: D5, J1, Q2, R3, R5, R9
